File: board/de0-extender-pll/trig3_board_de0-nano - LTC6957.brd (EAGLE design)
At the start: 160 x 75 mm, 94 parts, among them J1 10118192-0002LF, J12 4p-2.54, J13 BU-SMB-V, J17 2p-2.54, J23 2p-2.54, J24 2p-2.54, J32 2p-2.54, J34 2p-2.54, J38 2p-2.54, J42 2p-2.54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

Commit message: one change to silkscreen; added 4.7 uF capacitors to 3.3V header connections
Parts:
- added C14, C15: 4.7 uF, rcl:C0603
Connections:
- net 3V3: now also C14.1, C15.1
- net GND: now also C14.2, C15.2
Routing:
- net 3V3: track 61.8 -> 71.0 mm
Other:
- board text added: "+ALT CLOCK-"
- board text removed: "ALT CLOCK"
Changed lines of the file:
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@@
 <layers>
 <layer number="1" name="Top" color="4" fill="1" visible="yes" active="yes"/>
-<layer number="2" name="Route2" color="1" fill="3" visible="no" active="yes"/>
+<layer number="2" name="Route2" color="1" fill="3" visible="yes" active="yes"/>
 <layer number="3" name="Route3" color="4" fill="3" visible="no" active="no"/>
 <layer number="4" name="Route4" color="1" fill="4" visible="no" active="no"/>
@@
 <layer number="13" name="Route13" color="4" fill="5" visible="no" active="no"/>
 <layer number="14" name="Route14" color="1" fill="6" visible="no" active="no"/>
-<layer number="15" name="Route15" color="4" fill="6" visible="no" active="yes"/>
-<layer number="16" name="Bottom" color="1" fill="1" visible="no" active="yes"/>
+<layer number="15" name="Route15" color="4" fill="6" visible="yes" active="yes"/>
+<layer number="16" name="Bottom" color="1" fill="1" visible="yes" active="yes"/>
 <layer number="17" name="Pads" color="2" fill="1" visible="yes" active="yes"/>
 <layer number="18" name="Vias" color="2" fill="1" visible="yes" active="yes"/>
-<layer number="19" name="Unrouted" color="6" fill="1" visible="no" active="yes"/>
-<layer number="20" name="Dimension" color="24" fill="1" visible="no" active="yes"/>
+<layer number="19" name="Unrouted" color="6" fill="1" visible="yes" active="yes"/>
+<layer number="20" name="Dimension" color="24" fill="1" visible="yes" active="yes"/>
 <layer number="21" name="tPlace" color="7" fill="1" visible="yes" active="yes"/>
-<layer number="22" name="bPlace" color="7" fill="1" visible="no" active="yes"/>
-<layer number="23" name="tOrigins" color="15" fill="1" visible="no" active="yes"/>
-<layer number="24" name="bOrigins" color="15" fill="1" visible="no" active="yes"/>
+<layer number="22" name="bPlace" color="7" fill="1" visible="yes" active="yes"/>
+<layer number="23" name="tOrigins" color="15" fill="1" visible="yes" active="yes"/>
+<layer number="24" name="bOrigins" color="15" fill="1" visible="yes" active="yes"/>
 <layer number="25" name="tNames" color="7" fill="1" visible="yes" active="yes"/>
-<layer number="26" name="bNames" color="7" fill="1" visible="no" active="yes"/>
-<layer number="27" name="tValues" color="7" fill="1" visible="yes" active="yes"/>
+<layer number="26" name="bNames" color="7" fill="1" visible="yes" active="yes"/>
+<layer number="27" name="tValues" color="7" fill="1" visible="no" active="yes"/>
 <layer number="28" name="bValues" color="7" fill="1" visible="no" active="yes"/>
-<layer number="29" name="tStop" color="7" fill="3" visible="yes" active="yes"/>
+<layer number="29" name="tStop" color="7" fill="3" visible="no" active="yes"/>
 <layer number="30" name="bStop" color="7" fill="6" visible="no" active="yes"/>
-<layer number="31" name="tCream" color="7" fill="4" visible="yes" active="yes"/>
+<layer number="31" name="tCream" color="7" fill="4" visible="no" active="yes"/>
 <layer number="32" name="bCream" color="7" fill="5" visible="no" active="yes"/>
 <layer number="33" name="tFinish" color="6" fill="3" visible="no" active="yes"/>
@@
 <layer number="37" name="tTest" color="7" fill="1" visible="no" active="yes"/>
 <layer number="38" name="bTest" color="7" fill="1" visible="no" active="yes"/>
-<layer number="39" name="tKeepout" color="4" fill="11" visible="no" active="yes"/>
-<layer number="40" name="bKeepout" color="1" fill="11" visible="no" active="yes"/>
-<layer number="41" name="tRestrict" color="4" fill="10" visible="no" active="yes"/>
-<layer number="42" name="bRestrict" color="1" fill="10" visible="no" active="yes"/>
+<layer number="39" name="tKeepout" color="4" fill="11" visible="yes" active="yes"/>
+<layer number="40" name="bKeepout" color="1" fill="11" visible="yes" active="yes"/>
+<layer number="41" name="tRestrict" color="4" fill="10" visible="yes" active="yes"/>
+<layer number="42" name="bRestrict" color="1" fill="10" visible="yes" active="yes"/>
 <layer number="43" name="vRestrict" color="2" fill="10" visible="no" active="yes"/>
 <layer number="44" name="Drills" color="7" fill="1" visible="no" active="yes"/>
@@
 <layer number="50" name="dxf" color="7" fill="1" visible="no" active="no"/>
 <layer number="51" name="tDocu" color="7" fill="1" visible="yes" active="yes"/>
-<layer number="52" name="bDocu" color="7" fill="1" visible="no" active="yes"/>
+<layer number="52" name="bDocu" color="7" fill="1" visible="yes" active="yes"/>
 <layer number="53" name="tGND_GNDA" color="7" fill="9" visible="no" active="no"/>
 <layer number="54" name="bGND_GNDA" color="1" fill="9" visible="no" active="no"/>
@@
 <text x="-19.651" y="38.174" size="1.778" layer="21">+LASER CLOCK-</text>
 <text x="-38.4" y="60.96" size="1.778" layer="21">DIFF I/O PAIR</text>
-<text x="-16.238" y="62.857" size="1.778" layer="21">ALT CLOCK</text>
+<text x="-17.508" y="63.365" size="1.778" layer="21">+ALT CLOCK-</text>
 <wire x1="-45" y1="36" x2="-45" y2="111" width="0.1524" layer="20"/>
 <wire x1="-45" y1="111" x2="115" y2="111" width="0.1524" layer="20"/>
@@
 <attribute name="STANDARD" value="Manufacturer Recommendations" x="35.814" y="40.132" size="1.27" layer="27" display="off"/>
 </element>
+<element name="C14" library="rcl" library_urn="urn:adsk.eagle:library:334" package="C0603" package3d_urn="urn:adsk.eagle:package:23616/2" value="4.7 uF" x="12.065" y="92.71" smashed="yes" rot="R90">
+<attribute name="LCSC_PART#" value="C19666" x="12.065" y="92.71" size="1.27" layer="27" rot="R90" display="off"/>
+<attribute name="NAME" x="14.605" y="91.694" size="1.27" layer="25" rot="R90"/>
+<attribute name="POPULARITY" value="73" x="12.065" y="92.71" size="1.27" layer="27" rot="R90" display="off"/>
+<attribute name="SPICEPREFIX" value="C" x="12.065" y="92.71" size="1.27" layer="27" rot="R90" display="off"/>
+<attribute name="VALUE" x="13.97" y="92.075" size="1.27" layer="27" rot="R90"/>
+</element>
+<element name="C15" library="rcl" library_urn="urn:adsk.eagle:library:334" package="C0603" package3d_urn="urn:adsk.eagle:package:23616/2" value="4.7 uF" x="56.134" y="67.691" smashed="yes">
+<attribute name="LCSC_PART#" value="C19666" x="56.134" y="67.691" size="1.27" layer="27" display="off"/>
+<attribute name="NAME" x="54.483" y="65.278" size="1.27" layer="25"/>
+<attribute name="POPULARITY" value="73" x="56.134" y="67.691" size="1.27" layer="27" display="off"/>
+<attribute name="SPICEPREFIX" value="C" x="56.134" y="67.691" size="1.27" layer="27" display="off"/>
+<attribute name="VALUE" x="55.499" y="65.786" size="1.27" layer="27"/>
+</element>
 </elements>
 <signals>
@@
 <wire x1="30.861" y1="40.007" x2="30.861" y2="40.005" width="0.127" layer="1"/>
 <via x="30.861" y="40.005" extent="1-16" drill="0.35"/>
+<contactref element="C14" pad="2"/>
+<contactref element="C15" pad="2"/>
 </signal>
 <signal name="5V" class="1">
@@
 <wire x1="-17.30375" y1="97.94875" x2="-26.9875" y2="97.94875" width="0.127" layer="1"/>
 <wire x1="-27.78125" y1="97.155" x2="-27.85" y2="97" width="0.127" layer="1"/>
+<contactref element="C14" pad="1"/>
+<contactref element="C15" pad="1"/>
+<wire x1="49.73" y1="68.87" x2="50.909" y2="67.691" width="0.254" layer="1"/>
+<wire x1="50.909" y1="67.691" x2="55.284" y2="67.691" width="0.254" layer="1"/>
+<wire x1="8.97" y1="91.73" x2="11.935" y2="91.73" width="0.254" layer="1"/>
+<wire x1="11.935" y1="91.73" x2="12.065" y2="91.86" width="0.254" layer="1"/>
 </signal>
 <signal name="GPIO_024_C9">

Commit message: changed via hole size to reduce costs
Routing:
- net GPIO_113_P9: track 129.7 -> 128.8 mm
